File: Motor Controllers/KiCad/Motor Controllers.kicad_pcb (KiCad board)
At the start: 2 copper layers, 106 x 65 mm, 29 parts, among them J1 Conn_02x03_Counter_Clockwise, J2 Conn_02x03_Counter_Clockwise, J3 Conn_02x03_Counter_Clockwise, J4 Conn_02x03_Counter_Clockwise, J5 Power + I2C, U1 DRV8870DDA, U2 DRV8870DDA, U3 DRV8870DDA, U4 DRV8870DDA

Commit message: added encoders, slightly adjusted copper tracks
Routing:
- net +5V: track 319.9 -> 321.1 mm
- net GND: track 1.00 -> 0.00 mm, vias 828 -> 827
