File: Motor Controllers/KiCad/Motor Controllers.kicad_sch (KiCad schematic)
At the start: 9 parts, among them J1 Conn_02x03_Counter_Clockwise, J2 Conn_02x03_Counter_Clockwise, J3 Conn_02x03_Counter_Clockwise, J4 Conn_02x03_Counter_Clockwise, J5 Power + I2C

Commit message: added encoders, slightly adjusted copper tracks
Changed lines of the file:
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@@
   (junction (at 87.63 57.15) (diameter 0) (color 0 0 0 0)
   )
-  (junction (at 158.75 152.4) (diameter 0) (color 0 0 0 0)
-  )
   (junction (at 67.945 46.99) (diameter 0) (color 0 0 0 0)
   )
@@
   (junction (at 67.945 60.96) (diameter 0) (color 0 0 0 0)
   )
+  (junction (at 158.75 152.4) (diameter 0) (color 0 0 0 0)
+  )
+  (junction (at 133.35 152.4) (diameter 0) (color 0 0 0 0)
+  )
   (wire (pts (xy 57.15 106.68) (xy 64.77 106.68))
     (stroke (width 0) (type default))
@@
     (stroke (width 0) (type default))
   )
+  (wire (pts (xy 133.35 152.4) (xy 158.75 152.4))
+    (stroke (width 0) (type default))
+  )
   (wire (pts (xy 168.91 113.03) (xy 186.69 113.03))
     (stroke (width 0) (type default))
@@
     (stroke (width 0) (type default))
   )
-  (wire (pts (xy 158.75 152.4) (xy 158.75 153.67))
-    (stroke (width 0) (type default))
-  )
   (wire (pts (xy 106.68 88.265) (xy 106.68 113.665))
     (stroke (width 0) (type default))
@@
     )
   )
+  (text_box "J1,...,J4 : Digikey PPTC032LFBN-RC\nJ5 : Digikey SFH11-PBPC-D07-ST-BK"
+    (at 45.72 166.37 0) (size 36.83 4.445)
+    (stroke (width 0) (type default))
+    (fill (type none))
+    (effects (font (size 1 1) bold) (justify left top))
+  )
   (text "Mounting Holes" (at 102.87 162.56 0)
     (effects (font (size 2.5 2.5) (thickness 0.5) bold italic (color 0 0 0 1)) (justify left bottom))
@@
         )
       )
-    )
-  )
-  (symbol (lib_id "power:GND") (at 158.75 153.67 0) (unit 1)
-    (in_bom yes) (on_board yes) (dnp no) (fields_autoplaced)
-    (property "Reference" "#PWR08" (at 158.75 160.02 0)
-      (effects (font (size 1.27 1.27)) hide)
-    )
-    (property "Value" "GND" (at 158.75 158.75 0)
-      (effects (font (size 1.27 1.27)) hide)
-    )
-    (property "Footprint" "" (at 158.75 153.67 0)
-      (effects (font (size 1.27 1.27)) hide)
-    )
-    (property "Datasheet" "" (at 158.75 153.67 0)
-      (effects (font (size 1.27 1.27)) hide)
-    )
-    (pin "1")
-    (instances
-      (project "RoverPCB"
-        (path "/052e469e-2ccb-400e-bf36-44a19a932360/d5d68e58-4b58-44b0-923a-bd07b7aae5f3"
-          (reference "#PWR08") (unit 1)
-        )
-      )
-      (project "Power Supply"
-        (path "/c3cddd23-9147-41f9-a63c-fa9cc2f58832"
-          (reference "#PWR013") (unit 1)
-        )
-      )
-      (project "Motor Controllers"
-        (path "/df74bcb7-070d-4415-8f90-e15292cb5734"
-          (reference "#PWR025") (unit 1)
-        )
-      )
