File: Power Supply/Kicad/Power Supply.kicad_pcb (KiCad board)
At the start: 2 copper layers, 41 x 33.5 mm, 27 parts, among them J1 Conn_02x05_Counter_Clockwise, J2 PJ-082BH, U1 LM62440-Q1

Commit message: added encoders, slightly adjusted copper tracks
Parts:
- added TP1: TestPoint_Alt, TestPoint:TestPoint_Pad_2.0x2.0mm, F.Cu at (146.2, 96.5)
- added TP2: TestPoint_Alt, TestPoint:TestPoint_Pad_2.0x2.0mm, F.Cu at (152.8, 124.8)
Routing:
- net GND: vias 168 -> 166
Changed lines of the file:
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@@
       (sketchpadsonfab false)
       (subtractmaskfromsilk true)
-      (outputformat 4)
+      (outputformat 1)
       (mirror false)
       (drillshape 0)
@@
     )
   )
+  (footprint "TestPoint:TestPoint_Pad_2.0x2.0mm" (layer "F.Cu")
+    (at 152.75 124.75)
+    (descr "SMD rectangular pad as test Point, square 2.0mm side length")
+    (tags "test point SMD pad rectangle square")
+    (property "Sheetfile" "Power Supply.kicad_sch")
+    (property "Sheetname" "")
+    (property "ki_description" "test point (alternative shape)")
+    (property "ki_keywords" "test point tp")
+    (attr exclude_from_pos_files)
+    (fp_text reference "TP2" (at 0 -1.998) (layer "F.SilkS") hide
+        (effects (font (size 1 1) (thickness 0.15)))
+    )
+    (fp_text value "TestPoint_Alt" (at 0 2.05) (layer "F.Fab")
+        (effects (font (size 1 1) (thickness 0.15)))
+    )
+    (fp_text user "${REFERENCE}" (at 0 -2) (layer "F.Fab")
+        (effects (font (size 1 1) (thickness 0.15)))
+    )
+    (fp_line (start -1.2 -1.2) (end 1.2 -1.2)
+      (stroke (width 0.12) (type solid)) (layer "F.SilkS"))
+    (fp_line (start -1.2 1.2) (end -1.2 -1.2)
+      (stroke (width 0.12) (type solid)) (layer "F.SilkS"))
+    (fp_line (start 1.2 -1.2) (end 1.2 1.2)
+      (stroke (width 0.12) (type solid)) (layer "F.SilkS"))
+    (fp_line (start 1.2 1.2) (end -1.2 1.2)
+      (stroke (width 0.12) (type solid)) (layer "F.SilkS"))
+    (fp_line (start -1.5 -1.5) (end -1.5 1.5)
+      (stroke (width 0.05) (type solid)) (layer "F.CrtYd"))
+    (fp_line (start -1.5 -1.5) (end 1.5 -1.5)
+      (stroke (width 0.05) (type solid)) (layer "F.CrtYd"))
+    (fp_line (start 1.5 1.5) (end -1.5 1.5)
+      (stroke (width 0.05) (type solid)) (layer "F.CrtYd"))
+    (fp_line (start 1.5 1.5) (end 1.5 -1.5)
+      (stroke (width 0.05) (type solid)) (layer "F.CrtYd"))
+    (pad "1" smd rect (at 0 0) (size 2 2) (layers "F.Cu" "F.Mask")
+      (net 3 "+5V") (pinfunction "1") (pintype "passive"))
+  )
   (footprint "MountingHole:MountingHole_2.2mm_M2_ISO7380_Pad" (layer "F.Cu")
     (at 131.5 123.5)
@@
     (property "ki_keywords" "cap capacitor")
     (attr smd)
-    (fp_text reference "C12" (at 0 -2.75) (layer "F.SilkS")
+    (fp_text reference "C12" (at 0 -2) (layer "F.SilkS")
         (effects (font (size 1 1) (thickness 0.15)))
     )
@@
     )
   )
+  (footprint "TestPoint:TestPoint_Pad_2.0x2.0mm" (layer "F.Cu")
+    (at 146.25 96.5)
+    (descr "SMD rectangular pad as test Point, square 2.0mm side length")
+    (tags "test point SMD pad rectangle square")
+    (property "Sheetfile" "Power Supply.kicad_sch")
+    (property "Sheetname" "")
+    (property "ki_description" "test point (alternative shape)")
+    (property "ki_keywords" "test point tp")
+    (attr exclude_from_pos_files)
+    (fp_text reference "TP1" (at 0 -1.998) (layer "F.SilkS") hide
+        (effects (font (size 1 1) (thickness 0.15)))
+    )
+    (fp_text value "TestPoint_Alt" (at 0 2.05) (layer "F.Fab")
+        (effects (font (size 1 1) (thickness 0.15)))
+    )
+    (fp_text user "${REFERENCE}" (at 0 -2) (layer "F.Fab")
+        (effects (font (size 1 1) (thickness 0.15)))
+    )
+    (fp_line (start -1.2 -1.2) (end 1.2 -1.2)
+      (stroke (width 0.12) (type solid)) (layer "F.SilkS"))
+    (fp_line (start -1.2 1.2) (end -1.2 -1.2)
+      (stroke (width 0.12) (type solid)) (layer "F.SilkS"))
+    (fp_line (start 1.2 -1.2) (end 1.2 1.2)
+      (stroke (width 0.12) (type solid)) (layer "F.SilkS"))
+    (fp_line (start 1.2 1.2) (end -1.2 1.2)
+      (stroke (width 0.12) (type solid)) (layer "F.SilkS"))
+    (fp_line (start -1.5 -1.5) (end -1.5 1.5)
+      (stroke (width 0.05) (type solid)) (layer "F.CrtYd"))
+    (fp_line (start -1.5 -1.5) (end 1.5 -1.5)
+      (stroke (width 0.05) (type solid)) (layer "F.CrtYd"))
+    (fp_line (start 1.5 1.5) (end -1.5 1.5)
+      (stroke (width 0.05) (type solid)) (layer "F.CrtYd"))
+    (fp_line (start 1.5 1.5) (end 1.5 -1.5)
+      (stroke (width 0.05) (type solid)) (layer "F.CrtYd"))
+    (pad "1" smd rect (at 0 0) (size 2 2) (layers "F.Cu" "F.Mask")
+      (net 1 "+BATT") (pinfunction "1") (pintype "passive"))
+  )
   (footprint "Resistor_SMD:R_0402_1005Metric" (layer "F.Cu")
     (at 157.475 117.99 90)
@@
   (via (at 168.5 117.5) (size 0.7) (drill 0.3) (layers "F.Cu" "B.Cu") (free) (net 2))
   (via (at 168.5 112.5) (size 0.7) (drill 0.3) (layers "F.Cu" "B.Cu") (free) (net 2))
-  (via (at 141 104) (size 0.7) (drill 0.3) (layers "F.Cu" "B.Cu") (free) (net 2))
   (via (at 139 107) (size 0.7) (drill 0.3) (layers "F.Cu" "B.Cu") (free) (net 2))
   (via (at 168.5 101.5) (size 0.7) (drill 0.3) (layers "F.Cu" "B.Cu") (free) (net 2))
@@
   (via (at 131.5 117.5) (size 0.7) (drill 0.3) (layers "F.Cu" "B.Cu") (free) (net 2))
   (via (at 167 121) (size 0.7) (drill 0.3) (layers "F.Cu" "B.Cu") (free) (net 2))
-  (via (at 142 105) (size 0.7) (drill 0.3) (layers "F.Cu" "B.Cu") (free) (net 2))
+  (via (at 142 105.25) (size 0.7) (drill 0.3) (layers "F.Cu" "B.Cu") (free) (net 2))
   (via (at 145.5 118.5) (size 0.7) (drill 0.3) (layers "F.Cu" "B.Cu") (free) (net 2))
   (via (at 135.5 113.5) (size 0.7) (drill 0.3) (layers "F.Cu" "B.Cu") (free) (net 2))
@@
   (via (at 143.5 118.5) (size 0.7) (drill 0.3) (layers "F.Cu" "B.Cu") (free) (net 2))
   (via (at 144.5 119) (size 0.7) (drill 0.3) (layers "F.Cu" "B.Cu") (free) (net 2))
-  (via (at 142 104) (size 0.7) (drill 0.3) (layers "F.Cu" "B.Cu") (free) (net 2))
   (via (at 168.5 119.5) (size 0.7) (drill 0.3) (layers "F.Cu" "B.Cu") (free) (net 2))
   (via (at 145.4 108.1) (size 0.8) (drill 0.4) (layers "F.Cu" "B.Cu") (free) (net 2))
@@
   (segment (start 139.515 102.975) (end 139.475 102.935) (width 0.2) (layer "F.Cu") (net 3))
   (segment (start 139.365 105.025) (end 139.465 104.925) (width 0.5) (layer "F.Cu") (net 3))
-  (via (at 138.9 124.4) (size 0.8) (drill 0.4) (layers "F.Cu" "B.Cu") (net 3))
+  (via (at 138.9 125.25) (size 0.8) (drill 0.4) (layers "F.Cu" "B.Cu") (net 3))
   (via (at 152.475 105.45) (size 0.8) (drill 0.4) (layers "F.Cu" "B.Cu") (net 3))
   (via (at 151.25 123) (size 0.8) (drill 0.4) (layers "F.Cu" "B.Cu") (net 3))
   (via (at 148.125 105.675) (size 0.8) (drill 0.4) (layers "F.Cu" "B.Cu") (net 3))
   (via (at 138.275 105.025) (size 0.8) (drill 0.4) (layers "F.Cu" "B.Cu") (net 3))
-  (via (at 154.1 124) (size 0.8) (drill 0.4) (layers "F.Cu" "B.Cu") (net 3))
-  (segment (start 138.9 109.275) (end 137.525 107.9) (width 0.5) (layer "B.Cu") (net 3))
+  (via (at 154.1 123) (size 0.8) (drill 0.4) (layers "F.Cu" "B.Cu") (net 3))
+  (segment (start 137.525 105.775) (end 138.275 105.025) (width 0.5) (layer "B.Cu") (net 3))
+  (segment (start 138.9 125.25) (end 138.9 109.275) (width 0.5) (layer "B.Cu") (net 3))
+  (segment (start 154.1 123) (end 154.1 107.075) (width 0.5) (layer "B.Cu") (net 3))
   (segment (start 137.525 107.9) (end 137.525 105.775) (width 0.5) (layer "B.Cu") (net 3))
-  (segment (start 154.1 124) (end 154.1 107.075) (width 0.5) (layer "B.Cu") (net 3))
-  (segment (start 138.9 124.4) (end 138.9 109.275) (width 0.5) (layer "B.Cu") (net 3))
   (segment (start 151.25 123) (end 151.25 108.8) (width 0.5) (layer "B.Cu") (net 3))
-  (segment (start 154.1 107.075) (end 152.475 105.45) (width 0.5) (layer "B.Cu") (net 3))
+  (segment (start 138.9 109.275) (end 137.525 107.9) (width 0.5) (layer "B.Cu") (net 3))
   (segment (start 151.25 108.8) (end 148.125 105.675) (width 0.5) (layer "B.Cu") (net 3))
-  (segment (start 137.525 105.775) (end 138.275 105.025) (width 0.5) (layer "B.Cu") (net 3))
+  (segment (start 154.1 107.075) (end 152.475 105.45) (width 0.5) (layer "B.Cu") (net 3))
   (segment (start 141.045 101.75) (end 139.64 101.75) (width 0.2) (layer "F.Cu") (net 4))
   (segment (start 139.64 101.75) (end 139.475 101.915) (width 0.2) (layer "F.Cu") (net 4))
@@
       )
     )
+  )
+  (zone (net 1) (net_name "+BATT") (layer "F.Cu") (name "+VBATT") (hatch edge 0.5)
+    (priority 4)
+    (connect_pads yes (clearance 0.3))
+    (min_thickness 0.25) (filled_areas_thickness no)
+    (fill yes (thermal_gap 0.5) (thermal_bridge_width 0.5))
+    (polygon
+      (pts
+        (xy 144.5 94.75)
+        (xy 148 94.75)
+        (xy 148 98.25)
+        (xy 144.5 98.25)
+        (xy 144.5 96.75)
+      )
+    )
